File: 87C51.kicad_sch (KiCad schematic)
At the start: 18 parts, among them J8 68000-220HLF, J9 68000-220HLF, U1 87C51

Commit message: updated schematic after library re-organization
Parts:
- removed J8, J9: 68000-220HLF, Connector_PinHeader_2.54mm:PinHeader_1x20_P2.54mm_Vertical, symbol tutorial_2_library:VERT_HDR_20_2.54mm
- removed U1: 87C51, Package_LCC:PLCC-44_THT-Socket, symbol tutorial_2_library:87C51_Socket
- added J8, J9: 68000-220HLF, Connector_PinHeader_2.54mm:PinHeader_1x20_P2.54mm_Vertical, symbol NAE_Connectors:VERT_HDR_20_2.54mm
- added U1: 87C51, Package_LCC:PLCC-44_THT-Socket, symbol NAE_Integrated_Circuits:87C51_Socket
Connections:
- net 51_RESET: now also J9.9, U1.10 (RESET)
- net 51_RX: now also J9.10, U1.11 (P3.0/RxD)
- net 51_TX: now also J9.11, U1.13 (P3.1/TxD)
- net ALE/PROG: now also J8.11, U1.33 (ALE/~{PROG})
- net EA/VPP: now also J8.10, U1.35 (~{EA}/VPP)
- net GND: now also J9.20, U1.22 (GND)
- net LED1: now also J8.15, U1.29 (P2.5/A13)
- net LED2: now also J8.16, U1.28 (P2.4/A12)
- net M0: now also J9.13, U1.15 (P3.3/~{INT1})
- net M1: now also J9.14, U1.16 (P3.4/T0)
- net M2: now also J9.15, U1.17 (P3.5/T1)
- net P2.6: now also J8.14, U1.30 (P2.6/A14)
- net P2.7: now also J8.13, J8.20, U1.24 (P2.0/A8), U1.31 (P2.7/A15)
- net P3.6: now also J9.16, U1.18 (P3.6/~{WR})
- net P3.7: now also J9.17, U1.19 (P3.7/~{RD})
- net PA0: now also J9.1, U1.2 (P1.0/T2)
- net PA1: now also J9.2, U1.3 (P1.1/T2EX)
- net PA10: now also J8.18, U1.26 (P2.2/A10)
- net PA11: now also J8.17, U1.27 (P2.3/A11)
- net PA2: now also J9.3, U1.4 (P1.2)
- net PA3: now also J9.4, U1.5 (P1.3)
- net PA4: now also J9.5, U1.6 (P1.4)
- net PA5: now also J9.6, U1.7 (P1.5)
- net PA6: now also J9.7, U1.8 (P1.6)
- net PA7: now also J9.8, U1.9 (P1.7)
- net PA9: now also J8.19, U1.25 (P2.1/A9)
- net PD0: now also J8.2, U1.43 (P0.0/AD0)
- net PD1: now also J8.3, U1.42 (P0.1/AD1)
- net PD2: now also J8.4, U1.41 (P0.2/AD2)
- net PD3: now also J8.5, U1.40 (P0.3/AD3)
- net PD4: now also J8.6, U1.39 (P0.4/AD4)
- net PD5: now also J8.7, U1.38 (P0.5/AD5)
- net PD6: now also J8.8, U1.37 (P0.6/AD6)
- net PD7: now also J8.9, U1.36 (P0.7/AD7)
- net PSEN: now also J8.12, U1.32 (~{PSEN})
- net SHUNTL: now also J8.1, U1.44 (VCC)
- net at R14.2: now also J9.19, U1.21 (XTAL1)
- new net: J9.12, U1.14 (P3.2/~{INT0})
- new net: J9.18, U1.20 (XTAL2)
