File: CW312T_Connections.kicad_sch (KiCad schematic)
At the start: 6 parts, among them J11 1x3 straight header pins, P1 PCIEx4 EDGE CONNECTOR

Commit message: updated schematic after library re-organization
Parts:
- removed J11: 1x3 straight header pins, Connector_PinHeader_2.54mm:PinHeader_1x03_P2.54mm_Vertical, symbol tutorial_2_library:VERT_HDR_3_2.54mm
- removed JP1: ~, Jumper:SolderJumper-2_P1.3mm_Bridged2Bar_Pad1.0x1.5mm, symbol tutorial_2_library:Solder_Jumper_2_NC
- removed P1: PCIEx4 EDGE CONNECTOR, tutorial_2_library:CW312_Template, symbol tutorial_2_library:CW312T-Template
- added J11: 1x3 straight header pins, Connector_PinHeader_2.54mm:PinHeader_1x03_P2.54mm_Vertical, symbol NAE_Connectors:VERT_HDR_3_2.54mm
- added JP1: ~, Jumper:SolderJumper-2_P1.3mm_Bridged2Bar_Pad1.0x1.5mm, symbol NAE_Connectors:Solder_Jumper_2_NC
- added P1: PCIEx4 EDGE CONNECTOR, tutorial_2_library:CW312_Template, symbol NAE_Connectors:CW312T-Template
Connections:
- net AVR_RST: now also P1.B14 (nRST)
- net CLK: now also P1.B27 (CLKOUT)
- net GND: now also P1.A1 (GND), P1.A2 (GND), P1.A20 (GND), P1.A27 (GND), P1.A28 (GND), P1.A8 (GND), P1.B15 (GND), P1.B21 (GND), P1.B22 (GND), P1.B3 (GND), P1.B9 (GND)
- net GPIO3: now also P1.B18 (GPIO3)
- net GPIO4: now also P1.B19 (GPIO4)
- net LED1: now also P1.B11 (LED1)
- net LED2: now also P1.B12 (LED2)
- net LED3: now also P1.B13 (LED3)
- net M0: now also P1.A9 (HDR1)
- net M1: now also P1.A11 (HDR3)
- net M2: now also P1.A13 (HDR5)
- net MISO: now also P1.B23 (MISO)
- net MOSI: now also P1.B24 (MOSI)
- net RX: now also P1.B17 (GPIO2/RX)
- net SCK: now also P1.B20 (SCK)
- net SHUNTH: now also P1.A3 (FILT_LP), P1.B2 (SHUNTH), P1.B4 (FILT_HP)
- net SHUNTL: now also P1.B1 (SHUNTL)
- net TX: now also P1.B16 (GPIO1/TX)
- net VCC: now also J11.2, JP1.1, P1.A10 (HDR2), P1.A12 (HDR4), P1.A14 (HDR6), P1.B10 (IOVREF), P1.B5 (FILTIN)
- new net: J11.1, P1.A6 (VCC5.0)
- new net: J11.3, JP1.2, P1.A5 (VCC3.3)
